Commit message: Restyled environment

File: lenny_with_ros/motoman/motoman_sda10f_support/urdf/environment_macro.xacro (robot description, xacro)
@@ -1,4 +1,4 @@
 <?xml version="1.0" ?>
-<robot xmlns:xacro="http://ros.org/wiki/xacro">
+<model xmlns:xacro="http://ros.org/wiki/xacro">
 	<xacro:macro name="environment" params="name prefix">
 		<!-- link list -->
@@ -6,11 +6,30 @@
 		<visual>
 			<geometry>
-				<mesh filename="package://motoman_sda10f_support/meshes/environment/conveyor.STL"/>
+				<mesh filename="package://motoman_sda10f_support/meshes/environment/conveyor.stl" scale="0.01 0.01 0.01"/>
 				<!--IF .STL IS IN mm DUE SOLIDWORKS CONFLICT USE: scale="0.001 0.001 0.001" in mesh line-->
 			</geometry>
 			<origin xyz="0 0 0"/>
-			<material name="blue">
-				<color rgba="255 69 30 0.9"/>
+			<material name="gray_conveyor">
+				<texture filename="package://motoman_sda10f_support/meshes/environment/textures/silver.png"/>
+				<!--color rgba="${240/255} ${240/255} ${240/255} 1"/-->
 			</material>
+		</visual>
+</link>
+	<link name="feeder_table">
+		<visual>
+			<geometry>
+				<mesh filename="package://motoman_sda10f_support/meshes/environment/feeder_table.stl" scale="0.01 0.01 0.01"/>
+			</geometry>
+			<origin xyz="0 0 0"/>
+			<material name="gray_conveyor"/>
+		</visual>
+</link>
+	<link name="feeder_table_2">
+		<visual>
+			<geometry>
+				<mesh filename="package://motoman_sda10f_support/meshes/environment/feeder_table.stl" scale="0.01 0.01 0.01"/>
+			</geometry>
+			<origin xyz="0 0 0"/>
+			<material name="gray_conveyor"/>
 		</visual>
 </link>
@@ -21,6 +40,7 @@
 			</geometry>
 			<origin xyz="-0.615 0 -0.76"/>
-			<material name="blue">
-				<color rgba="255 69 30 0.9"/>
+			<material name="beige_table">
+				<!--color rgba="${249/255} ${226/255} ${211/255} 1"/-->
+				<texture filename="package://motoman_sda10f_support/meshes/environment/textures/beige.png"/>
 			</material>
 		</visual>
@@ -30,9 +50,8 @@
 			<geometry>
 				<mesh filename="package://motoman_sda10f_support/meshes/environment/worktable.STL" scale="0.001 0.001 0.001"/>
-				<!--IF .STL IS IN mm DUE SOLIDWORKS CONFLICT USE: scale="0.001 0.001 0.001" in mesh line-->
 			</geometry>
 			<origin xyz="-0.625 0 0"/>
-			<material name="blue">
-				<color rgba="255 69 30 0.9"/>
+			<material name="gray_worktable">
+				<color rgba="${45/255} ${135/255} ${149/255} 1"/>
 			</material>
 		</visual>
@@ -44,6 +63,6 @@
 			</geometry>
 			<origin xyz="-0.035 0 -0.035"/>
-			<material name="blue">
-				<color rgba="255 69 30 0.9"/>
+			<material name="yellow_beacon">
+				<color rgba="${255/255} ${255/255} ${0/255} 1"/>
 			</material>
 		</visual>
@@ -66,15 +85,42 @@
 			</geometry>
 			<origin xyz="-0.7 0 -1.40"/>
-			<material name="blue">
-				<color rgba="255 69 30 0.9"/>
+			<material name="festo">
+				<texture filename="package://motoman_sda10f_support/meshes/environment/textures/aqua.png"/>
 			</material>
 		</visual>
+		<collision>
+				<geometry>
+					<mesh filename="package://motoman_sda10f_support/meshes/environment/MPS.STL" />
+				</geometry>
+				<origin xyz= "-0.7 0 -1.40"/>
+		</collision>
 </link>
+	<!--link name="MPS_FAKE">
+		<visual>
+			<geometry>
+				<mesh filename="package://motoman_sda10f_support/meshes/environment/MPS_FAKE.stl" scale="0.008 0.008 0.008"/>
+			</geometry>
+			<origin xyz="0 0 0"/>
+			<material name="cyan_mps">
+				<color rgba="${168/255} ${224/255} ${198/255} 1"/>
+			</material>
+		</visual>
+</link-->
 		<!-- joint list -->
 	<joint name="coveyor_to_robot" type="fixed">
 		<parent link="torso_base_link"/>
 		<child link="conveyor"/>
-		<origin xyz="-2.92 -2.45 0.13" rpy="0 0 -1.571"/>
-				<!--WRITE 0.4 IN Z IF THE ROBOT IS AT THE SAME HEIGHT OF THE CONVEYOR-->
+		<!--origin xyz="-2.92 -2.45 0.13" rpy="0 0 -1.571"/-->
+		<origin xyz="0.618 -1.244 -0.252" rpy="0 0 -1.571"/>
+	</joint>
+	<joint name="feeder_table_to_robot" type="fixed">
+		<parent link="torso_base_link"/>
+		<child link="feeder_table"/>
+		<origin xyz="0.05 0.47 -0.3" rpy="0 0 1.5708"/>
+	</joint>
+	<joint name="feeder_table_2_to_robot" type="fixed">
+		<parent link="feeder_table"/>
+		<child link="feeder_table_2"/>
+		<origin xyz="1.11 0 0" rpy="0 0 0"/>
 	</joint>
 	<joint name="table_to_robot" type="fixed">
@@ -103,6 +149,11 @@
 		<origin xyz="-0.111 -1.405 -0.3" rpy="1.571 0 1.571"/> <!--Sumo 5cm a las MPS por si acaso-->
 	</joint>
+		<!--joint name="MPS_FAKE_to_robot" type="fixed">
+		<parent link="torso_base_link"/>
+		<child link="MPS_FAKE"/>
+		<origin xyz="-1.35 0.6 -0.3" rpy="0 0 -1.5708"/--> <!--Sumo 5cm a las MPS por si acaso-->
+	<!--/joint-->
 		<!-- end of joint list -->
 	</xacro:macro>
 	<xacro:environment name="environment" prefix="environment_"/>
-</robot>
+</model>

File: lenny_with_ros/motoman/motoman_sda10f_support/urdf/kinect_macro.xacro (robot description, xacro)
@@ -1,4 +1,4 @@
 <?xml version="1.0" ?>
-<robot xmlns:xacro="http://ros.org/wiki/xacro">
+<model xmlns:xacro="http://ros.org/wiki/xacro">
 	<xacro:macro name="kinect" params="name prefix">
 		<!-- link list -->
@@ -9,6 +9,6 @@
 			</geometry>
 			<origin xyz="-0.14 0 0"/>
-			<material name="black">
-				<color rgba="176 176 176 0.9"/>
+			<material name="green_kinect">
+				<color rgba="${68/255} ${218/255} ${63/255} 1"/>
 			</material>
 		</visual>
@@ -18,7 +18,4 @@
 				</geometry>
 				<origin xyz= "-0.16 0 0"/>
-				<material name="black">
-					<color rgba="176 176 176 0.9"/>
-				</material>
 		</collision>
 	</link>
@@ -29,6 +26,6 @@
 			</geometry>
 			<origin xyz="-0.14 0 0"/>
-			<material name="black">
-				<color rgba="176 176 176 0.9"/>
+			<material name="orange_kinect">
+				<color rgba="${244/255} ${94/255} ${0/255} 1"/>
 			</material>
 		</visual>
@@ -44,5 +41,5 @@
 		<parent link="torso_base_link"/>
 		<child link="base_kinect"/>
-		<origin xyz="0.894 0.056 2.09" rpy="1.54 0 -1.52"/> <!--origin xyz="0.148 0.845 1.6425" rpy="1.54 0 -3.14"/> <ESTA ES LA TRANSFORMADA QUE HAY QUE MEDIR menos 30cm en Z-->
+		<origin xyz="0.817 0.056 2.07" rpy="1.54 0 -1.52"/> <!--origin xyz="0.148 0.845 1.6425" rpy="1.54 0 -3.14"/> <ESTA ES LA TRANSFORMADA QUE HAY QUE MEDIR menos 30cm en Z-->
 	</joint>
 	<joint name="base_kinect_to_kinect" type="fixed">
@@ -54,3 +51,3 @@
 	</xacro:macro>
 	<xacro:kinect name="kinect" prefix="kinect_"/>
-</robot>
+</model>

File: lenny_with_ros/motoman/motoman_sda10f_support/urdf/sda10f.xacro (robot description, xacro)
@@ -2,6 +2,4 @@
 <robot name="motoman_sda10f" xmlns:xacro="http://ros.org/wiki/xacro">
 	<xacro:include filename="$(find motoman_sda10f_support)/urdf/sda10f_macro.xacro" />
-	<xacro:include filename="$(find motoman_sda10f_support)/urdf/kinect_macro.xacro" />
-	<xacro:include filename="$(find motoman_sda10f_support)/urdf/environment_macro.xacro"/>
 	<xacro:motoman_sda10f prefix=""/>
 </robot>

File: lenny_with_ros/motoman/motoman_sda10f_support/urdf/sda10f_macro.xacro (robot description, xacro)
@@ -3,4 +3,8 @@
      <xacro:include filename="$(find motoman_sda10f_support)/urdf/common_torso_macro.xacro" />
      <xacro:include filename="$(find motoman_sda10f_support)/urdf/arm_macro.xacro" />
+     <xacro:include filename="$(find robotiq_c2_model_visualization)/urdf/robotiq_c2_model_macro.xacro"/>
+     <xacro:include filename="$(find motoman_sda10f_support)/urdf/kinect_macro.xacro" />
+	<xacro:include filename="$(find motoman_sda10f_support)/urdf/environment_macro.xacro"/>
+	<xacro:include filename="$(find motoman_sda10f_support)/urdf/visual_environment_macro.xacro"/>
      <xacro:macro name="motoman_sda10f" params="prefix">
         <xacro:torso name="${prefix}torso" prefix="${prefix}torso_"/>
@@ -11,9 +15,15 @@
             <origin xyz="0.09996 -0.0275 0.32214" rpy="1.57 0 0" />
         </xacro:motoman_arm>
+        <xacro:robotiq_c2_model prefix=""/>
+        	<joint name="left_gripper_to_robot" type="fixed">
+			<parent link="${prefix}arm_left_link_tool0" />
+			<child link = "${prefix}robotiq_85_adapter_link" />
+			<origin xyz="0 0 0" rpy="0 1.5708 -0.7854" />
+		</joint>
      </xacro:macro>
 <!-- The following xacro is kept for backwards compatibility, it should not be used -->
 <!-- see: https://github.com/ros-industrial/motoman/issues/166 -->
-     <xacro:macro name="sda10f">
+     <!--xacro:macro name="sda10f">
           <xacro:motoman_sda10f prefix=""/>
-     </xacro:macro>
+     </xacro:macro-->
 </robot>
